File: PCBs/ECESD/GSP RevC.kicad_sch (KiCad schematic)
At the start: 3 parts

Commit message: Changed PCB 1
Parts:
- removed H1, H2, H3: MountingHole, MountingHole:MountingHole_2.2mm_M2, symbol Mechanical:MountingHole
- added H100, H101: MountingHole, MountingHole:MountingHole_2.2mm_M2, symbol Mechanical:MountingHole
Changed lines of the file:
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@@
 	(title_block
 		(title "Motion Board")
-		(date "2025-01-13")
-		(rev "B")
+		(date "2025-02-02")
+		(rev "C")
 		(company "GlideSense Pro")
 		(comment 1 "Josue Cavazos Jr.")
+		(comment 2 "Andrew Thomas")
 	)
 	(text "[2] MCU"
 		(exclude_from_sim no)
-		(at 121.666 68.326 0)
-		(effects
-			(font
-				(size 5.0038 5.0038)
-				(thickness 1.0008)
-				(bold yes)
-				(italic yes)
-			)
-			(justify left bottom)
+		(at 130.302 71.628 0)
+		(effects
+			(font
+				(size 5 5)
+				(bold yes)
+				(italic yes)
+			)
+		)
+	)
+	(text "[3] Motion"
+		(exclude_from_sim no)
+		(at 221.234 71.628 0)
+		(effects
+			(font
+				(size 5 5)
+				(bold yes)
+				(italic yes)
+			)
+		)
+	)
+	(text "Motion Board"
+		(exclude_from_sim no)
+		(at 53.34 26.67 0)
+		(effects
+			(font
+				(size 6 6)
+				(thickness 1.2)
+				(bold yes)
+				(italic yes)
+			)
 		)
 	)
 	(text "[1] Power"
 		(exclude_from_sim no)
-		(at 50.292 67.818 0)
-		(effects
-			(font
-				(size 5.0038 5.0038)
-				(thickness 1.0008)
-				(bold yes)
-				(italic yes)
-			)
-			(justify left bottom)
-		)
-	)
-	(text "Motion Board"
-		(exclude_from_sim no)
-		(at 18.288 27.432 0)
-		(effects
-			(font
-				(size 6 6)
-				(thickness 1.0008)
-				(bold yes)
-				(italic yes)
-			)
-			(justify left bottom)
-		)
-	)
-	(text "[3] Motion"
-		(exclude_from_sim no)
-		(at 192.786 68.326 0)
-		(effects
-			(font
-				(size 5.0038 5.0038)
-				(thickness 1.0008)
-				(bold yes)
-				(italic yes)
-			)
-			(justify left bottom)
+		(at 49.022 71.374 0)
+		(effects
+			(font
+				(size 5 5)
+				(bold yes)
+				(italic yes)
+			)
 		)
 	)
 	(symbol
 		(lib_id "Mechanical:MountingHole")
-		(at 21.59 179.07 0)
+		(at 21.59 173.99 0)
 		(unit 1)
 		(exclude_from_sim yes)
@@
 		(dnp no)
 		(fields_autoplaced yes)
-		(property "Reference" "H2"
-			(at 24.13 177.7999 0)
+		(property "Reference" "H100"
+			(at 24.13 172.7199 0)
 			(effects
 				(font
@@
 		)
 		(property "Value" "MountingHole"
-			(at 24.13 180.3399 0)
+			(at 24.13 175.2599 0)
 			(effects
 				(font
@@
 		)
 		(property "Footprint" "MountingHole:MountingHole_2.2mm_M2"
-			(at 21.59 179.07 0)
+			(at 21.59 173.99 0)
 			(effects
 				(font
@@
 		)
 		(property "Datasheet" "~"
-			(at 21.59 179.07 0)
+			(at 21.59 173.99 0)
 			(effects
 				(font
@@
 		)
 		(property "Description" "Mounting Hole without connection"
-			(at 21.59 179.07 0)
-			(effects
-				(font
-					(size 1.27 1.27)
-				)
-				(hide yes)
-			)
-		)
-		(instances
-			(project "GlideSensePro MIII"
-				(path "/78dae1b0-3dec-4f9a-bc4d-7b6fb3842c26"
-					(reference "H2")
+			(at 21.59 173.99 0)
+			(effects
+				(font
+					(size 1.27 1.27)
+				)
+				(hide yes)
+			)
+		)
+		(instances
+			(project "GSP RevC"
+				(path "/3a13d9bb-3700-499a-bcbc-99ebe364dcaa"
+					(reference "H100")
 					(unit 1)
 				)
@@
 	(symbol
 		(lib_id "Mechanical:MountingHole")
-		(at 21.59 172.72 0)
+		(at 21.59 180.34 0)
 		(unit 1)
 		(exclude_from_sim yes)
@@
 		(dnp no)
 		(fields_autoplaced yes)
-		(property "Reference" "H1"
-			(at 24.13 171.4499 0)
+		(property "Reference" "H101"
+			(at 24.13 179.0699 0)
 			(effects
 				(font
@@
 		)
 		(property "Value" "MountingHole"
-			(at 24.13 173.9899 0)
+			(at 24.13 181.6099 0)
 			(effects
 				(font
@@
 		)
 		(property "Footprint" "MountingHole:MountingHole_2.2mm_M2"
-			(at 21.59 172.72 0)
+			(at 21.59 180.34 0)
 			(effects
 				(font
@@
 		)
 		(property "Datasheet" "~"
-			(at 21.59 172.72 0)
+			(at 21.59 180.34 0)
 			(effects
 				(font
@@
 		)
 		(property "Description" "Mounting Hole without connection"
-			(at 21.59 172.72 0)
-			(effects
-				(font
-					(size 1.27 1.27)
-				)
-				(hide yes)
-			)
-		)
-		(instances
-			(project "GlideSensePro MIII"
-				(path "/78dae1b0-3dec-4f9a-bc4d-7b6fb3842c26"
-					(reference "H1")
+			(at 21.59 180.34 0)
+			(effects
+				(font
+					(size 1.27 1.27)
+				)
+				(hide yes)
+			)
+		)
+		(instances
+			(project "GSP RevC"
+				(path "/3a13d9bb-3700-499a-bcbc-99ebe364dcaa"
+					(reference "H101")
 					(unit 1)
 				)
@@
 		)
 	)
-	(symbol
-		(lib_id "Mechanical:MountingHole")
-		(at 21.59 185.42 0)
-		(unit 1)
-		(exclude_from_sim yes)
-		(in_bom no)
-		(on_board yes)
-		(dnp no)
-		(fields_autoplaced yes)
-		(property "Reference" "H3"
-			(at 24.13 184.1499 0)
-			(effects
-				(font
-					(size 1.27 1.27)
-				)
-				(justify left)
-			)
-		)
-		(property "Value" "MountingHole"
-			(at 24.13 186.6899 0)
-			(effects
-				(font
-					(size 1.27 1.27)
-				)
-				(justify left)
-			)
-		)
-		(property "Footprint" "MountingHole:MountingHole_2.2mm_M2"
-			(at 21.59 185.42 0)
-			(effects
-				(font
-					(size 1.27 1.27)
-				)
-				(hide yes)
-			)
-		)
-		(property "Datasheet" "~"
-			(at 21.59 185.42 0)
-			(effects
-				(font
-					(size 1.27 1.27)
-				)
-				(hide yes)
-			)
-		)
-		(property "Description" "Mounting Hole without connection"
-			(at 21.59 185.42 0)
-			(effects
-				(font
-					(size 1.27 1.27)
-				)
-				(hide yes)
-			)
-		)
-		(instances
-			(project "GlideSensePro MIII"
-				(path "/78dae1b0-3dec-4f9a-bc4d-7b6fb3842c26"
-					(reference "H3")
-					(unit 1)
-				)
-			)
-		)
-	)
 	(sheet
-		(at 121.92 80.01)
-		(size 58.42 57.15)
+		(at 201.93 82.55)
+		(size 69.85 62.23)
 		(fields_autoplaced yes)
 		(stroke
@@
 			(color 0 0 0 0.0000)
 		)
-		(property "Sheetname" "MCU"
-			(at 121.92 79.2984 0)
+		(property "Sheetname" "Motion"
+			(at 201.93 81.8384 0)
 			(effects
 				(font
@@
 			)
 		)
-		(property "Sheetfile" "MCU.kicad_sch"
-			(at 121.92 137.7446 0)
+		(property "Sheetfile" "Motion.kicad_sch"
+			(at 201.93 145.3646 0)
 			(effects
 				(font
@@
 		)
 		(instances
-			(project "GlideSensePro MIII"
-				(path "/78dae1b0-3dec-4f9a-bc4d-7b6fb3842c26"
-					(page "3")
+			(project "GSP RevC"
+				(path "/3a13d9bb-3700-499a-bcbc-99ebe364dcaa"
+					(page "4")
 				)
 			)
@@
 	)
 	(sheet
-		(at 50.8 80.01)
-		(size 58.42 57.15)
+		(at 30.48 82.55)
+		(size 69.85 62.23)
 		(fields_autoplaced yes)
 		(stroke
@@
 		)
 		(property "Sheetname" "Power"
-			(at 50.8 79.2984 0)
+			(at 30.48 81.8384 0)
 			(effects
 				(font
@@
 		)
 		(property "Sheetfile" "Power.kicad_sch"
-			(at 50.8 137.7446 0)
+			(at 30.48 145.3646 0)
 			(effects
 				(font
@@
 		)
 		(instances
-			(project "GlideSensePro MIII"
-				(path "/78dae1b0-3dec-4f9a-bc4d-7b6fb3842c26"
+			(project "GSP RevC"
+				(path "/3a13d9bb-3700-499a-bcbc-99ebe364dcaa"
 					(page "2")
 				)
@@
 	)
 	(sheet
-		(at 193.04 80.01)
-		(size 58.42 57.15)
+		(at 115.57 82.55)
+		(size 69.85 62.23)
 		(fields_autoplaced yes)
 		(stroke
@@
 			(color 0 0 0 0.0000)
 		)
-		(property "Sheetname" "Motion"
-			(at 193.04 79.2984 0)
+		(property "Sheetname" "MCU"
+			(at 115.57 81.8384 0)
 			(effects
 				(font
@@
 			)
 		)
-		(property "Sheetfile" "Motion.kicad_sch"
-			(at 193.04 137.7446 0)
+		(property "Sheetfile" "MCU.kicad_sch"
+			(at 115.57 145.3646 0)
 			(effects
 				(font
@@
 		)
 		(instances
-			(project "GlideSensePro MIII"
-				(path "/78dae1b0-3dec-4f9a-bc4d-7b6fb3842c26"
-					(page "4")
-				)
-			)
+			(project "GSP RevC"
+				(path "/3a13d9bb-3700-499a-bcbc-99ebe364dcaa"
+					(page "3")
+				)
+			)
